Commit message: Set gripper position closed by default

File: hand_e_gripper_description/urdf/hand_e_gripper.urdf.xacro (robot description, xacro)
@@ -56,6 +56,6 @@
         <joint name="${prefix}_finger_left_joint" type="prismatic">
             <limit lower="0.0" upper="0.025" effort="1.0" velocity="0.0125"/>
-            <axis xyz="0 -1 0"/>
-            <origin xyz="0 0.028 0.0995" rpy="0 0 0" />
+            <axis xyz="0 1 0"/>
+            <origin xyz="0 0.003 0.0995" rpy="0 0 0" />
             <parent link="${prefix}_base_link"/>
             <child link="${prefix}_left_finger" />
@@ -104,6 +104,6 @@
         <joint name="${prefix}_finger_right_joint" type="prismatic">
             <limit lower="0.0" upper="0.025" effort="1.0" velocity="0.0125"/>
-            <axis xyz="0 1 0"/>
-            <origin xyz="0 -0.028 0.0995" rpy="0 0 0" />
+            <axis xyz="0 -1 0"/>
+            <origin xyz="0 -0.003 0.0995" rpy="0 0 0" />
             <parent link="${prefix}_base_link"/>
             <child link="${prefix}_right_finger" />
